File: AM32电调.kicad_sch (KiCad schematic)
At the start: 74 parts, among them Q1 IRF7480M, Q2 IRF7480M, Q3 IRF7480M, Q4 IRF7480M, Q5 IRF7480M, Q6 IRF7480M, U1 STM32G071GBUxN, U3 AP2210K-3.3TRG1, U4 INA199xxDCK

Commit message: ADD: final draft
Parts:
- removed U4: INA199xxDCK, Package_TO_SOT_SMD:SOT-363_SC-70-6, symbol Amplifier_Current:INA199xxDCK
- added U8: INA240A1PW, Package_SO:TSSOP-8_4.4x3mm_P0.65mm, symbol Amplifier_Current:INA240A1PW
- R1, R10, R11, R12, R13, R14, R15, R16, R18, R19, R2, R20, R21, R22, R23, R24, R25, R26, R27, R28, R29, R3, R30, R31, R4, R6, R7, R8, R9: footprint Resistor_SMD_AKL:R_0402_1005Metric_Pad0.72x0.64mm -> Resistor_SMD:R_0402_1005Metric
- R17: value 47k -> 4.7k; footprint Resistor_SMD_AKL:R_0402_1005Metric_Pad0.72x0.64mm -> Resistor_SMD:R_0402_1005Metric
Connections:
- net +3.3V: now also U8.5 (V+)
- net ADC_CUR: now also U7.4, U7.5; no longer U7.1, U7.6
- net GND: now also U7.1, U7.6, U8.1 (GND), U8.4 (GND), U8.6 (REF2), U8.7 (REF1); no longer U7.4, U7.5
- net VBAT: now also U8.2 (+)
- net VM: now also U8.3 (-)
- net at R30.2: now also U7.3; no longer U7.2
- net at R31.2: now also U7.2; no longer U7.3
- net at R6.1: now also U8.8
